File: pcb/shell/shell.kicad_pcb (KiCad board)
At the start: 2 copper layers, 343.2 x 114.4 mm, 126 parts, among them J1 Conn_01x15, J2 Conn_01x15

Commit message: updated pcb edge cut
Other:
- outline, holes or cut-outs redrawn

Commit message: fixed per key rgb
Parts:
- added D62: LED, LED_SMD:LED_SK6812_PLCC4_5.0x5.0mm_P3.2mm, B.Cu at (210.7, 83.3)
- added D63: LED, LED_SMD:LED_SK6812_PLCC4_5.0x5.0mm_P3.2mm, B.Cu at (210.7, 89.9)
- added D64: LED, LED_SMD:LED_SK6812_PLCC4_5.0x5.0mm_P3.2mm, B.Cu at (210.7, 96.5)
- added D65: LED, LED_SMD:LED_SK6812_PLCC4_5.0x5.0mm_P3.2mm, B.Cu at (210.7, 103.1)
- added D66: LED, LED_SMD:LED_SK6812_PLCC4_5.0x5.0mm_P3.2mm, B.Cu at (210.7, 109.7)
- added D67: LED, LED_SMD:LED_SK6812_PLCC4_5.0x5.0mm_P3.2mm, B.Cu at (202.3, 83.3)
- added D68: LED, LED_SMD:LED_SK6812_PLCC4_5.0x5.0mm_P3.2mm, B.Cu at (202.3, 89.9)
- added D69: LED, LED_SMD:LED_SK6812_PLCC4_5.0x5.0mm_P3.2mm, B.Cu at (202.3, 96.5)
- added D70: LED, LED_SMD:LED_SK6812_PLCC4_5.0x5.0mm_P3.2mm, B.Cu at (202.3, 103.1)
- added D71: LED, LED_SMD:LED_SK6812_PLCC4_5.0x5.0mm_P3.2mm, B.Cu at (202.3, 109.7)
- added D72: LED, LED_SMD:LED_SK6812_PLCC4_5.0x5.0mm_P3.2mm, B.Cu at (193.9, 83.3)
- added D73: LED, LED_SMD:LED_SK6812_PLCC4_5.0x5.0mm_P3.2mm, B.Cu at (193.9, 89.9)
- added D74: LED, LED_SMD:LED_SK6812_PLCC4_5.0x5.0mm_P3.2mm, B.Cu at (193.9, 96.5)
- added D75: LED, LED_SMD:LED_SK6812_PLCC4_5.0x5.0mm_P3.2mm, B.Cu at (193.9, 103.1)
- added D76: LED, LED_SMD:LED_SK6812_PLCC4_5.0x5.0mm_P3.2mm, B.Cu at (193.9, 109.7)
- added D77: LED, LED_SMD:LED_SK6812_PLCC4_5.0x5.0mm_P3.2mm, B.Cu at (185.5, 83.3)
- added D78: LED, LED_SMD:LED_SK6812_PLCC4_5.0x5.0mm_P3.2mm, B.Cu at (185.5, 89.9)
- added D79: LED, LED_SMD:LED_SK6812_PLCC4_5.0x5.0mm_P3.2mm, B.Cu at (185.5, 96.5)
- added D80: LED, LED_SMD:LED_SK6812_PLCC4_5.0x5.0mm_P3.2mm, B.Cu at (185.5, 103.1)
- added LED1: LED, PCM_marbastlib-mx:LED_MX_6028R-ROT, B.Cu at (65.1, 141.6)
- added LED10: LED, PCM_marbastlib-mx:LED_MX_6028R-ROT, B.Cu at (289.7, 144.3)
- added LED11: LED, PCM_marbastlib-mx:LED_MX_6028R-ROT, B.Cu at (309.3, 141.6)
- added LED12: LED, PCM_marbastlib-mx:LED_MX_6028R-ROT, B.Cu at (328.4, 141.6)
- added LED13: LED, PCM_marbastlib-mx:LED_MX_6028R, B.Cu at (56.3, 160.7)
- added LED14: LED, PCM_marbastlib-mx:LED_MX_6028R, B.Cu at (80.1, 160.7)
- added LED15: LED, PCM_marbastlib-mx:LED_MX_6028R, B.Cu at (99.8, 163.0)
- added LED16: LED, PCM_marbastlib-mx:LED_MX_6028R, B.Cu at (118.4, 166.9)
- added LED17: LED, PCM_marbastlib-mx:LED_MX_6028R, B.Cu at (137.1, 170.9)
- added LED18: LED, PCM_marbastlib-mx:LED_MX_6028R, B.Cu at (155.7, 174.8)
- added LED19: LED, PCM_marbastlib-mx:LED_MX_6028R, B.Cu at (237.8, 174.8)
- added LED2: LED, PCM_marbastlib-mx:LED_MX_6028R-ROT, B.Cu at (84.2, 141.6)
- added LED20: LED, PCM_marbastlib-mx:LED_MX_6028R, B.Cu at (256.4, 170.8)
- added LED21: LED, PCM_marbastlib-mx:LED_MX_6028R, B.Cu at (275.0, 166.9)
- added LED22: LED, PCM_marbastlib-mx:LED_MX_6028R, B.Cu at (293.7, 162.9)
- added LED23: LED, PCM_marbastlib-mx:LED_MX_6028R, B.Cu at (313.4, 160.7)
- added LED24: LED, PCM_marbastlib-mx:LED_MX_6028R, B.Cu at (337.2, 160.7)
- added LED25: LED, PCM_marbastlib-mx:LED_MX_6028R-ROT, B.Cu at (49.9, 179.7)
- added LED26: LED, PCM_marbastlib-mx:LED_MX_6028R-ROT, B.Cu at (76.0, 179.7)
- added LED27: LED, PCM_marbastlib-mx:LED_MX_6028R-ROT, B.Cu at (95.8, 181.6)
- added LED28: LED, PCM_marbastlib-mx:LED_MX_6028R-ROT, B.Cu at (114.5, 185.5)
- added LED29: LED, PCM_marbastlib-mx:LED_MX_6028R-ROT, B.Cu at (133.1, 189.5)
- added LED3: LED, PCM_marbastlib-mx:LED_MX_6028R-ROT, B.Cu at (103.8, 144.3)
- added LED30: LED, PCM_marbastlib-mx:LED_MX_6028R-ROT, B.Cu at (151.7, 193.5)
- added LED31: LED, PCM_marbastlib-mx:LED_MX_6028R-ROT, B.Cu at (241.7, 193.4)
- added LED32: LED, PCM_marbastlib-mx:LED_MX_6028R-ROT, B.Cu at (260.4, 189.5)
- added LED33: LED, PCM_marbastlib-mx:LED_MX_6028R-ROT, B.Cu at (279.0, 185.5)
- added LED34: LED, PCM_marbastlib-mx:LED_MX_6028R-ROT, B.Cu at (297.6, 181.6)
- added LED35: LED, PCM_marbastlib-mx:LED_MX_6028R-ROT, B.Cu at (317.5, 179.7)
- added LED36: LED, PCM_marbastlib-mx:LED_MX_6028R-ROT, B.Cu at (343.7, 179.7)
- added LED37: LED, PCM_marbastlib-mx:LED_MX_6028R, B.Cu at (45.8, 198.8)
- added LED38: LED, PCM_marbastlib-mx:LED_MX_6028R, B.Cu at (71.9, 198.8)
- added LED39: LED, PCM_marbastlib-mx:LED_MX_6028R, B.Cu at (91.9, 200.2)
- added LED4: LED, PCM_marbastlib-mx:LED_MX_6028R-ROT, B.Cu at (122.4, 148.3)
- added LED40: LED, PCM_marbastlib-mx:LED_MX_6028R, B.Cu at (110.5, 204.2)
- added LED41: LED, PCM_marbastlib-mx:LED_MX_6028R, B.Cu at (129.2, 208.1)
- added LED42: LED, PCM_marbastlib-mx:LED_MX_6028R, B.Cu at (147.8, 212.1)
- added LED43: LED, PCM_marbastlib-mx:LED_MX_6028R, B.Cu at (245.7, 212.1)
- added LED44: LED, PCM_marbastlib-mx:LED_MX_6028R, B.Cu at (264.3, 208.1)
- added LED45: LED, PCM_marbastlib-mx:LED_MX_6028R, B.Cu at (283.0, 204.2)
- added LED46: LED, PCM_marbastlib-mx:LED_MX_6028R, B.Cu at (301.6, 200.2)
- added LED47: LED, PCM_marbastlib-mx:LED_MX_6028R, B.Cu at (321.5, 198.8)
- added LED48: LED, PCM_marbastlib-mx:LED_MX_6028R, B.Cu at (342.9, 198.8)
- added LED49: LED, PCM_marbastlib-mx:LED_MX_6028R, B.Cu at (364.4, 198.8)
- added LED5: LED, PCM_marbastlib-mx:LED_MX_6028R-ROT, B.Cu at (141.0, 152.2)
- added LED50: LED, PCM_marbastlib-mx:LED_MX_6028R-ROT, B.Cu at (41.8, 217.8)
- added LED51: LED, PCM_marbastlib-mx:LED_MX_6028R-ROT, B.Cu at (65.6, 217.8)
- added LED52: LED, PCM_marbastlib-mx:LED_MX_6028R-ROT, B.Cu at (87.9, 218.9)
- added LED53: LED, PCM_marbastlib-mx:LED_MX_6028R-ROT, B.Cu at (108.9, 223.3)
- added LED54: LED, PCM_marbastlib-mx:LED_MX_6028R-ROT, B.Cu at (141.5, 230.2)
- added LED55: LED, PCM_marbastlib-mx:LED_MX_6028R-ROT, B.Cu at (171.8, 236.7)
- added LED56: LED, PCM_marbastlib-mx:LED_MX_6028R-ROT, B.Cu at (221.7, 236.7)
- added LED57: LED, PCM_marbastlib-mx:LED_MX_6028R-ROT, B.Cu at (249.7, 230.7)
- added LED58: LED, PCM_marbastlib-mx:LED_MX_6028R-ROT, B.Cu at (279.9, 224.3)
- added LED59: LED, PCM_marbastlib-mx:LED_MX_6028R-ROT, B.Cu at (303.2, 219.3)
- added LED6: LED, PCM_marbastlib-mx:LED_MX_6028R-ROT, B.Cu at (159.7, 156.2)
- added LED60: LED, PCM_marbastlib-mx:LED_MX_6028R-ROT, B.Cu at (327.9, 217.8)
- added LED61: LED, PCM_marbastlib-mx:LED_MX_6028R-ROT, B.Cu at (354.1, 217.8)
- added LED7: LED, PCM_marbastlib-mx:LED_MX_6028R-ROT, B.Cu at (233.8, 156.2)
- added LED8: LED, PCM_marbastlib-mx:LED_MX_6028R-ROT, B.Cu at (252.4, 152.2)
- added LED9: LED, PCM_marbastlib-mx:LED_MX_6028R-ROT, B.Cu at (271.1, 148.3)
- J1, J2: value Conn_01x15 -> Conn_01x11; footprint Connector_PinHeader_2.54mm:PinHeader_1x15_P2.54mm_Vertical -> Connector_PinSocket_2.54mm:PinSocket_1x11_P2.54mm_Vertical
- moved J2 9.39 mm to (225.8, 190.1)
- moved J1 9.15 mm to (166.1, 190.0)
- moved D60 2.45 mm to (333.2, 216.9)
- moved D61 2.41 mm to (359.4, 216.9)
- moved D20 2.40 mm to (261.5, 168.8)
- moved D21 2.40 mm to (280.1, 164.8)
- moved D22 2.40 mm to (298.7, 160.9)
- moved D32 2.40 mm to (265.4, 187.4)
- moved D34 2.40 mm to (302.7, 179.5)
- moved D59 2.40 mm to (308.3, 217.3)
- moved D33 2.40 mm to (284.1, 183.5)
- moved D19 2.40 mm to (242.8, 172.7)
- moved D43 2.40 mm to (250.8, 210.0)
- moved D56 2.40 mm to (226.8, 234.6)
- moved D57 2.40 mm to (254.7, 228.6)
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Connections:
- net Net-(MX16-Pad1) renamed col3
- D1 pad 1: Net-(D1-K) -> row0
- D10 pad 1: Net-(D1-K) -> row0
- D11 pad 1: Net-(D1-K) -> row0
- D12 pad 1: Net-(D1-K) -> row0
- D13 pad 1: Net-(D13-K) -> row1
- D14 pad 1: Net-(D13-K) -> row1
- D15 pad 1: Net-(D13-K) -> row1
- D16 pad 1: Net-(D13-K) -> row1
- D17 pad 1: Net-(D13-K) -> row1
- D18 pad 1: Net-(D13-K) -> row1
- D19 pad 1: Net-(D13-K) -> row1
- D2 pad 1: Net-(D1-K) -> row0
- D20 pad 1: Net-(D13-K) -> row1
- D21 pad 1: Net-(D13-K) -> row1
- D22 pad 1: Net-(D13-K) -> row1
- D23 pad 1: Net-(D13-K) -> row1
- D24 pad 1: Net-(D13-K) -> row1
- D25 pad 1: Net-(D25-K) -> row2
- D26 pad 1: Net-(D25-K) -> row2
- D27 pad 1: Net-(D25-K) -> row2
- D28 pad 1: Net-(D25-K) -> row2
- D29 pad 1: Net-(D25-K) -> row2
- D3 pad 1: Net-(D1-K) -> row0
- D30 pad 1: Net-(D25-K) -> row2
- D31 pad 1: Net-(D25-K) -> row2
- D32 pad 1: Net-(D25-K) -> row2
- D33 pad 1: Net-(D25-K) -> row2
- D34 pad 1: Net-(D25-K) -> row2
- D35 pad 1: Net-(D25-K) -> row2
- D36 pad 1: Net-(D25-K) -> row2
- D37 pad 1: Net-(D37-K) -> row3
- D38 pad 1: Net-(D37-K) -> row3
- D39 pad 1: Net-(D37-K) -> row3
- D4 pad 1: Net-(D1-K) -> row0
- D40 pad 1: Net-(D37-K) -> row3
- D41 pad 1: Net-(D37-K) -> row3
- D42 pad 1: Net-(D37-K) -> row3
- D43 pad 1: Net-(D37-K) -> row3
- D44 pad 1: Net-(D37-K) -> row3
- D45 pad 1: Net-(D37-K) -> row3
- D46 pad 1: Net-(D37-K) -> row3
- D47 pad 1: Net-(D37-K) -> row3
- D48 pad 1: Net-(D37-K) -> row3
- D49 pad 1: Net-(D37-K) -> row5
- D5 pad 1: Net-(D1-K) -> row0
- D50 pad 1: Net-(D50-K) -> row4
- D51 pad 1: Net-(D50-K) -> row4
- D52 pad 1: Net-(D50-K) -> row4
- D53 pad 1: Net-(D50-K) -> row4
- D54 pad 1: Net-(D50-K) -> row4
- D55 pad 1: Net-(D50-K) -> row4
- D56 pad 1: Net-(D50-K) -> row4
- D57 pad 1: Net-(D50-K) -> row4
- D58 pad 1: Net-(D50-K) -> row4
- D59 pad 1: Net-(D50-K) -> row4
- D6 pad 1: Net-(D1-K) -> row0
- D60 pad 1: Net-(D50-K) -> row4
- D61 pad 1: Net-(D50-K) -> row4
- D7 pad 1: Net-(D1-K) -> row0
- D8 pad 1: Net-(D1-K) -> row0
- D9 pad 1: Net-(D1-K) -> row0
- J1 pad 1: unconnected-(J1-Pin_1-Pad1) -> perkey-rgb
- J1 pad 10: unconnected-(J1-Pin_10-Pad10) -> row3
- J1 pad 11: unconnected-(J1-Pin_11-Pad11) -> row4
- J1 pad 2: unconnected-(J1-Pin_2-Pad2) -> col0
- J1 pad 3: unconnected-(J1-Pin_3-Pad3) -> col1
- J1 pad 4: unconnected-(J1-Pin_4-Pad4) -> col2
- J1 pad 5: unconnected-(J1-Pin_5-Pad5) -> col4
- J1 pad 6: unconnected-(J1-Pin_6-Pad6) -> col5
- J1 pad 7: unconnected-(J1-Pin_7-Pad7) -> row0
- J1 pad 8: unconnected-(J1-Pin_8-Pad8) -> row1
- J1 pad 9: unconnected-(J1-Pin_9-Pad9) -> row2
- J2 pad 1: unconnected-(J2-Pin_1-Pad1) -> underglow-rgb
- J2 pad 10: unconnected-(J2-Pin_10-Pad10) -> GND
- J2 pad 2: unconnected-(J2-Pin_2-Pad2) -> col11
- J2 pad 3: unconnected-(J2-Pin_3-Pad3) -> col10
- J2 pad 4: unconnected-(J2-Pin_4-Pad4) -> col9
- J2 pad 5: unconnected-(J2-Pin_5-Pad5) -> col8
- J2 pad 6: unconnected-(J2-Pin_6-Pad6) -> col7
- J2 pad 7: unconnected-(J2-Pin_7-Pad7) -> col6
- J2 pad 8: unconnected-(J2-Pin_8-Pad8) -> row5
- J2 pad 9: unconnected-(J2-Pin_9-Pad9) -> VCC
- MX1 pad 1: Net-(MX1-Pad1) -> col0
- MX10 pad 1: Net-(MX10-Pad1) -> col9
- MX11 pad 1: Net-(MX11-Pad1) -> col10
- MX12 pad 1: Net-(MX12-Pad1) -> col11
- MX13 pad 1: Net-(MX1-Pad1) -> col0
- MX14 pad 1: Net-(MX14-Pad1) -> col1
- MX15 pad 1: Net-(MX15-Pad1) -> col2
- MX17 pad 1: Net-(MX17-Pad1) -> col4
- MX18 pad 1: Net-(MX18-Pad1) -> col5
- MX19 pad 1: Net-(MX19-Pad1) -> col6
- MX2 pad 1: Net-(MX14-Pad1) -> col1
- MX20 pad 1: Net-(MX20-Pad1) -> col7
- MX21 pad 1: Net-(MX21-Pad1) -> col8
- MX22 pad 1: Net-(MX10-Pad1) -> col9
- MX23 pad 1: Net-(MX11-Pad1) -> col10
- MX24 pad 1: Net-(MX12-Pad1) -> col11
- MX25 pad 1: Net-(MX1-Pad1) -> col0
- MX26 pad 1: Net-(MX14-Pad1) -> col1
- MX27 pad 1: Net-(MX15-Pad1) -> col2
- MX29 pad 1: Net-(MX17-Pad1) -> col4
- MX3 pad 1: Net-(MX15-Pad1) -> col2
- MX30 pad 1: Net-(MX18-Pad1) -> col5
- MX31 pad 1: Net-(MX19-Pad1) -> col6
- MX32 pad 1: Net-(MX20-Pad1) -> col7
- MX33 pad 1: Net-(MX21-Pad1) -> col8
- MX34 pad 1: Net-(MX10-Pad1) -> col9
- MX35 pad 1: Net-(MX11-Pad1) -> col10
- MX36 pad 1: Net-(MX12-Pad1) -> col11
- MX37 pad 1: Net-(MX1-Pad1) -> col0
- MX38 pad 1: Net-(MX14-Pad1) -> col1
- MX39 pad 1: Net-(MX15-Pad1) -> col2
- MX41 pad 1: Net-(MX17-Pad1) -> col4
- MX42 pad 1: Net-(MX18-Pad1) -> col5
- MX43 pad 1: Net-(MX19-Pad1) -> col6
- MX44 pad 1: Net-(MX20-Pad1) -> col7
- MX45 pad 1: Net-(MX21-Pad1) -> col8
- MX46 pad 1: Net-(MX10-Pad1) -> col9
- MX47 pad 1: Net-(MX11-Pad1) -> col10
- MX48 pad 1: Net-(MX12-Pad1) -> col11
- MX49 pad 1: unconnected-(MX49-Pad1) -> col0
- MX5 pad 1: Net-(MX17-Pad1) -> col4
- MX50 pad 1: Net-(MX1-Pad1) -> col0
- MX51 pad 1: Net-(MX14-Pad1) -> col1
- MX52 pad 1: Net-(MX15-Pad1) -> col2
- MX54 pad 1: Net-(MX17-Pad1) -> col4
- MX55 pad 1: Net-(MX18-Pad1) -> col5
- MX56 pad 1: Net-(MX19-Pad1) -> col6
- MX57 pad 1: Net-(MX20-Pad1) -> col7
- MX58 pad 1: Net-(MX21-Pad1) -> col8
- MX59 pad 1: Net-(MX10-Pad1) -> col9
- MX6 pad 1: Net-(MX18-Pad1) -> col5
- MX60 pad 1: Net-(MX11-Pad1) -> col10
- MX61 pad 1: Net-(MX12-Pad1) -> col11
- MX7 pad 1: Net-(MX19-Pad1) -> col6
- MX8 pad 1: Net-(MX20-Pad1) -> col7
- MX9 pad 1: Net-(MX21-Pad1) -> col8
Routing:
- net Net-(D1-K): track 212.7 -> 0.00 mm, vias 12 -> 0
- net Net-(D13-K): track 179.9 -> 0.00 mm, vias 12 -> 0
- net Net-(D25-K): track 153.9 -> 0.00 mm, vias 12 -> 0
- net Net-(D37-K): track 139.1 -> 0.00 mm, vias 13 -> 0
- net Net-(MX19-Pad1): track 103.6 -> 0.00 mm
- net Net-(MX18-Pad1): track 95.1 -> 0.00 mm
- net Net-(MX20-Pad1): track 87.2 -> 0.00 mm
- net Net-(MX12-Pad1): track 86.6 -> 0.00 mm
- net Net-(MX17-Pad1): track 85.5 -> 0.00 mm
- net Net-(MX1-Pad1): track 83.3 -> 0.00 mm
- net Net-(MX14-Pad1): track 82.8 -> 0.00 mm
- net Net-(MX11-Pad1): track 82.8 -> 0.00 mm
- net Net-(MX15-Pad1): track 80.1 -> 0.00 mm
- net col3: track 79.7 -> 0.00 mm
- net Net-(MX10-Pad1): track 79.5 -> 0.00 mm
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
Commit message: added underglow rgb
Parts:
- removed D62, D63, D64, D65, D67, D68, D69, D70, D71, D72, D73, D74, D75, D76, D77, D78, D79, D80: LED, LED_SMD:LED_SK6812_PLCC4_5.0x5.0mm_P3.2mm
- added UG10: LED, LED_SMD:LED_SK6812_PLCC4_5.0x5.0mm_P3.2mm, B.Cu at (317.6, 226.6)
- added UG11: LED, LED_SMD:LED_SK6812_PLCC4_5.0x5.0mm_P3.2mm, B.Cu at (294.8, 229.2)
- added UG12: LED, LED_SMD:LED_SK6812_PLCC4_5.0x5.0mm_P3.2mm, B.Cu at (270.8, 232.8)
- added UG13: LED, LED_SMD:LED_SK6812_PLCC4_5.0x5.0mm_P3.2mm, B.Cu at (234.6, 241.7)
- added UG14: LED, LED_SMD:LED_SK6812_PLCC4_5.0x5.0mm_P3.2mm, B.Cu at (206.1, 246.1)
- added UG15: LED, LED_SMD:LED_SK6812_PLCC4_5.0x5.0mm_P3.2mm, B.Cu at (185.5, 245.8)
- added UG16: LED, LED_SMD:LED_SK6812_PLCC4_5.0x5.0mm_P3.2mm, B.Cu at (156.7, 243.9)
- added UG17: LED, LED_SMD:LED_SK6812_PLCC4_5.0x5.0mm_P3.2mm, B.Cu at (120.1, 235.4)
- added UG18: LED, LED_SMD:LED_SK6812_PLCC4_5.0x5.0mm_P3.2mm, B.Cu at (94.7, 230.6)
- added UG19: LED, LED_SMD:LED_SK6812_PLCC4_5.0x5.0mm_P3.2mm, B.Cu at (77.6, 227.9)
- added UG2: LED, LED_SMD:LED_SK6812_PLCC4_5.0x5.0mm_P3.2mm, B.Cu at (258.1, 131.5)
- added UG20: LED, LED_SMD:LED_SK6812_PLCC4_5.0x5.0mm_P3.2mm, B.Cu at (54.6, 228.4)
- added UG21: LED, LED_SMD:LED_SK6812_PLCC4_5.0x5.0mm_P3.2mm, B.Cu at (24.8, 199.6)
- added UG22: LED, LED_SMD:LED_SK6812_PLCC4_5.0x5.0mm_P3.2mm, B.Cu at (25.3, 179.9)
- added UG23: LED, LED_SMD:LED_SK6812_PLCC4_5.0x5.0mm_P3.2mm, B.Cu at (28.2, 160.9)
- added UG24: LED, LED_SMD:LED_SK6812_PLCC4_5.0x5.0mm_P3.2mm, B.Cu at (73.8, 122.4)
- added UG25: LED, LED_SMD:LED_SK6812_PLCC4_5.0x5.0mm_P3.2mm, B.Cu at (96.7, 122.6)
- added UG26: LED, LED_SMD:LED_SK6812_PLCC4_5.0x5.0mm_P3.2mm, B.Cu at (117.1, 125.5)
- added UG27: LED, LED_SMD:LED_SK6812_PLCC4_5.0x5.0mm_P3.2mm, B.Cu at (134.5, 129.2)
- added UG28: LED, LED_SMD:LED_SK6812_PLCC4_5.0x5.0mm_P3.2mm, B.Cu at (154.0, 135.3)
- added UG3: LED, LED_SMD:LED_SK6812_PLCC4_5.0x5.0mm_P3.2mm, B.Cu at (277.4, 127.2)
- added UG4: LED, LED_SMD:LED_SK6812_PLCC4_5.0x5.0mm_P3.2mm, B.Cu at (304.2, 122.8)
- added UG5: LED, LED_SMD:LED_SK6812_PLCC4_5.0x5.0mm_P3.2mm, B.Cu at (319.0, 123.5)
- added UG6: LED, LED_SMD:LED_SK6812_PLCC4_5.0x5.0mm_P3.2mm, B.Cu at (355.6, 161.2)
- added UG7: LED, LED_SMD:LED_SK6812_PLCC4_5.0x5.0mm_P3.2mm, B.Cu at (365.1, 179.6)
- added UG8: LED, LED_SMD:LED_SK6812_PLCC4_5.0x5.0mm_P3.2mm, B.Cu at (381.7, 199.7)
- added UG9: LED, LED_SMD:LED_SK6812_PLCC4_5.0x5.0mm_P3.2mm, B.Cu at (343.3, 226.5)
- moved UG1 36.4 mm to (237.2, 134.7), turned to -168 degrees
- renumbered D66 to UG1
Routing:
- net Net-(LED7-DOUT): track 0.00 -> 0.61 mm

Commit message: started routing left side
Parts:
- moved UG26 41.3 mm to (108.1, 165.8)
- moved UG8 37.5 mm to (380.9, 162.2), turned to 102 degrees
- moved UG21 37.4 mm to (31.8, 236.3), turned to -78 degrees
- moved UG27 37.4 mm to (127.2, 165.8)
- moved UG22 37.2 mm to (28.3, 217.0), turned to -78 degrees
- moved UG23 36.9 mm to (27.2, 197.8), turned to -78 degrees
- moved D49 34.9 mm to (368.6, 162.9), turned to 102 degrees
- moved LED50 34.4 mm to (52.2, 250.6), turned to -168 degrees
- moved MX50 34.2 mm to (51.2, 245.6), turned to -168 degrees
- moved UG7 33.9 mm to (360.6, 146.0), turned to 102 degrees
- moved LED49 33.9 mm to (363.8, 164.9), turned to -168 degrees
- moved MX49 33.8 mm to (362.7, 159.9), turned to -168 degrees
- moved D61 33.4 mm to (362.7, 183.7), turned to 102 degrees
- moved D50 33.3 mm to (57.3, 248.6), turned to 102 degrees
- moved LED37 33.0 mm to (52.2, 231.1), turned to -168 degrees
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Routing:
- net col5: track 0.00 -> 110.6 mm
- net col4: track 0.00 -> 97.9 mm
- net col3: track 0.00 -> 88.5 mm
- net col2: track 0.00 -> 87.1 mm
- net Net-(LED53-DOUT): track 0.00 -> 28.5 mm
- net Net-(LED54-DOUT): track 0.00 -> 26.0 mm
- net Net-(UG25-DOUT): track 0.00 -> 20.4 mm
- net Net-(LED52-DOUT): track 0.00 -> 16.4 mm
- net Net-(UG26-DOUT): track 0.00 -> 16.1 mm, vias 0 -> 2
- net Net-(UG27-DOUT): track 0.00 -> 16.1 mm, vias 0 -> 2
- net Net-(LED27-DOUT): track 0.00 -> 14.1 mm
- net Net-(LED28-DOUT): track 0.00 -> 14.1 mm
- net Net-(LED29-DOUT): track 0.00 -> 14.1 mm
- net Net-(LED16-DIN): track 0.00 -> 14.1 mm
- net Net-(LED40-DIN): track 0.00 -> 14.1 mm
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Other:
- board size 343.2 x 114.4 mm -> 338.7 x 154.8 mm

Commit message: added a couple more traces on left side
Routing:
- net VCC: track 0.47 -> 385.6 mm, vias 0 -> 6
- net row4: track 0.00 -> 92.8 mm, vias 0 -> 3
- net row2: track 0.00 -> 77.8 mm, vias 0 -> 2
- net row0: track 0.00 -> 76.7 mm, vias 0 -> 2
- net row1: track 0.00 -> 75.4 mm
- net row3: track 0.00 -> 74.8 mm
- net Net-(UG16-DOUT): track 0.00 -> 41.7 mm, vias 0 -> 2
- net perkey-rgb: track 0.00 -> 25.3 mm
- net Net-(LED18-DIN): track 0.00 -> 21.8 mm
- net Net-(LED30-DOUT): track 0.00 -> 21.3 mm
- net Net-(UG18-DOUT): track 0.00 -> 19.8 mm
- net Net-(UG17-DOUT): track 0.00 -> 19.2 mm, vias 0 -> 2
- net Net-(LED51-DOUT): track 0.00 -> 9.45 mm
- net GND: track 0.00 -> 9.16 mm, vias 0 -> 1
- net Net-(LED2-DOUT): track 0.00 -> 7.77 mm
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