File: pcb/core/special/core.kicad_pcb (KiCad board)
At the start: 2 copper layers, 79.3 x 74.6 mm, 12 parts, among them J1 Conn_01x11, J2 Conn_01x11, J3 I2C, J4 SPI, U1 Helios

Commit message: added versions
Parts:
- added REF**: OSHW-Symbol_6.7x6mm_Copper, Symbol:OSHW-Symbol_6.7x6mm_Copper, F.Cu at (173.6, 162.7)
Other:
- board text added: "floookay.de/barnacle special core v1.0 CERN-OHL-S"
